File: LPC11UxxMini.sch (EAGLE design)
At the start: 37 parts, among them Q1 BC857B, U1 LPC11Uxx, U2 MCP1252-33X50I/MS, Y1 12MHz

Commit message: Squished to true Arduino Pro Mini form factor (Prototype 2)
also added pin_map.txt
Parts:
- added JP9: FIDUCIALUFIDUCIAL, SparkFun-Aesthetics:FIDUCIALUFIDUCIAL
- renumbered LED1 to POWER, LED2 to STATUS
Connections:
- net LED1_RESISTOR renamed POWER_LED_RESISTOR
- net LED2_RESISTOR renamed STATUS_LED_RESISTOR
Changed lines of the file:
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@@
 <?xml version="1.0" encoding="utf-8"?>
 <!DOCTYPE eagle SYSTEM "eagle.dtd">
-<eagle version="6.3">
+<eagle version="6.4">
 <drawing>
 <settings>
@@
 <layer number="97" name="Info" color="7" fill="1" visible="yes" active="yes"/>
 <layer number="98" name="Guide" color="6" fill="1" visible="yes" active="yes"/>
+<layer number="99" name="SpiceOrder" color="5" fill="1" visible="yes" active="yes"/>
 <layer number="100" name="Muster" color="7" fill="1" visible="yes" active="yes"/>
 <layer number="101" name="Patch_Top" color="12" fill="4" visible="yes" active="yes"/>
@@
 <part name="P+8" library="SparkFun-Aesthetics" deviceset="VCC" device=""/>
 <part name="U$2" library="logxen" deviceset="VIN" device=""/>
-<part name="LED2" library="microbuilder" deviceset="LED" device="0603_NOOUTLINE" value="20mA"/>
+<part name="STATUS" library="microbuilder" deviceset="LED" device="0603_NOOUTLINE" value="20mA"/>
 <part name="GND4" library="SparkFun-Aesthetics" deviceset="GND" device=""/>
-<part name="LED1" library="microbuilder" deviceset="LED" device="0603_NOOUTLINE" value="20mA"/>
+<part name="POWER" library="microbuilder" deviceset="LED" device="0603_NOOUTLINE" value="20mA"/>
 <part name="R1" library="SparkFun-Resistors" deviceset="RESISTOR" device="0402-RES" value="330 Ohm"/>
 <part name="R2" library="SparkFun-Resistors" deviceset="RESISTOR" device="0402-RES" value="200 Ohm"/>
@@
 <part name="R12" library="SparkFun-Resistors" deviceset="RESISTOR" device="0402-RES" value="10kOhm"/>
 <part name="P+7" library="SparkFun-Aesthetics" deviceset="VCC" device=""/>
+<part name="JP9" library="SparkFun-Aesthetics" deviceset="FIDUCIAL" device="UFIDUCIAL"/>
 </parts>
 <sheets>
@@
 <instance part="P+8" gate="1" x="190.5" y="0"/>
 <instance part="U$2" gate="G$1" x="248.92" y="111.76"/>
-<instance part="LED2" gate="G$1" x="30.48" y="17.78" rot="MR180"/>
+<instance part="STATUS" gate="G$1" x="30.48" y="17.78" rot="MR180"/>
 <instance part="GND4" gate="1" x="35.56" y="12.7"/>
-<instance part="LED1" gate="G$1" x="30.48" y="27.94" rot="MR180"/>
+<instance part="POWER" gate="G$1" x="30.48" y="27.94" rot="MR180"/>
 <instance part="R1" gate="G$1" x="17.78" y="27.94"/>
 <instance part="R2" gate="G$1" x="17.78" y="17.78"/>
@@
 <instance part="R12" gate="G$1" x="185.42" y="55.88" rot="R90"/>
 <instance part="P+7" gate="1" x="177.8" y="66.04"/>
+<instance part="JP9" gate="G$1" x="5.08" y="5.08"/>
 </instances>
 <busses>
@@
 <pinref part="GND4" gate="1" pin="GND"/>
 <wire x1="35.56" y1="27.94" x2="35.56" y2="17.78" width="0.1524" layer="91"/>
-<pinref part="LED2" gate="G$1" pin="C"/>
+<pinref part="STATUS" gate="G$1" pin="C"/>
 <wire x1="35.56" y1="17.78" x2="35.56" y2="15.24" width="0.1524" layer="91"/>
 <wire x1="33.02" y1="17.78" x2="35.56" y2="17.78" width="0.1524" layer="91"/>
-<pinref part="LED1" gate="G$1" pin="C"/>
+<pinref part="POWER" gate="G$1" pin="C"/>
 <wire x1="35.56" y1="27.94" x2="33.02" y2="27.94" width="0.1524" layer="91"/>
 <junction x="35.56" y="17.78"/>
@@
 </segment>
 </net>
-<net name="LED2_RESISTOR" class="0">
+<net name="STATUS_LED_RESISTOR" class="0">
 <segment>
 <pinref part="R2" gate="G$1" pin="2"/>
-<pinref part="LED2" gate="G$1" pin="A"/>
+<pinref part="STATUS" gate="G$1" pin="A"/>
 <wire x1="22.86" y1="17.78" x2="25.4" y2="17.78" width="0.1524" layer="91"/>
 </segment>
@@
 </segment>
 </net>
-<net name="LED1_RESISTOR" class="0">
+<net name="POWER_LED_RESISTOR" class="0">
 <segment>
 <pinref part="R1" gate="G$1" pin="2"/>
-<pinref part="LED1" gate="G$1" pin="A"/>
+<pinref part="POWER" gate="G$1" pin="A"/>
 <wire x1="22.86" y1="27.94" x2="25.4" y2="27.94" width="0.1524" layer="91"/>
 </segment>

Commit message: Added pull-down to P0_3 USB_VBUS
leaving P0_3 floating does not seem to reliably select serial
programming mode vs. usb programming mode, so a 10k pull-down was added
to assert serial mode when usb power is not present.
Parts:
- added R13: 10kOhm, SparkFun-Resistors:RESISTOR0402-RES
Connections:
- net GND: now also R13.1
- net MC_USB_VBUS: now also R13.2
Other:
- moved on the sheet: R10
Changed lines of the file:
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@@
 <?xml version="1.0" encoding="utf-8"?>
 <!DOCTYPE eagle SYSTEM "eagle.dtd">
-<eagle version="6.4">
+<eagle version="6.3">
 <drawing>
 <settings>
@@
 <part name="P+7" library="SparkFun-Aesthetics" deviceset="VCC" device=""/>
 <part name="JP9" library="SparkFun-Aesthetics" deviceset="FIDUCIAL" device="UFIDUCIAL"/>
+<part name="R13" library="SparkFun-Resistors" deviceset="RESISTOR" device="0402-RES" value="10kOhm"/>
 </parts>
 <sheets>
@@
 <instance part="R8" gate="G$1" x="116.84" y="5.08"/>
 <instance part="R9" gate="G$1" x="124.46" y="12.7" rot="R90"/>
-<instance part="R10" gate="G$1" x="78.74" y="7.62" rot="R90"/>
+<instance part="R10" gate="G$1" x="78.74" y="2.54" rot="R90"/>
 <instance part="GND5" gate="1" x="193.04" y="96.52"/>
 <instance part="GND6" gate="1" x="251.46" y="101.6"/>
@@
 <instance part="P+7" gate="1" x="177.8" y="66.04"/>
 <instance part="JP9" gate="G$1" x="5.08" y="5.08"/>
+<instance part="R13" gate="G$1" x="88.9" y="2.54" rot="R90"/>
 </instances>
 <busses>
@@
 <wire x1="99.06" y1="-25.4" x2="99.06" y2="-27.94" width="0.1524" layer="91"/>
 <junction x="99.06" y="-25.4"/>
+<pinref part="R13" gate="G$1" pin="1"/>
+<wire x1="88.9" y1="-2.54" x2="88.9" y2="-25.4" width="0.1524" layer="91"/>
+<wire x1="88.9" y1="-25.4" x2="99.06" y2="-25.4" width="0.1524" layer="91"/>
 </segment>
 </net>
@@
 <pinref part="R10" gate="G$1" pin="2"/>
 <pinref part="U1" gate="G$1" pin="PIO0_3/USB_VBUS"/>
+<wire x1="78.74" y1="7.62" x2="78.74" y2="12.7" width="0.1524" layer="91"/>
+<pinref part="R13" gate="G$1" pin="2"/>
 <wire x1="78.74" y1="12.7" x2="78.74" y2="25.4" width="0.1524" layer="91"/>
+<wire x1="78.74" y1="12.7" x2="88.9" y2="12.7" width="0.1524" layer="91"/>
+<wire x1="88.9" y1="12.7" x2="88.9" y2="7.62" width="0.1524" layer="91"/>
+<junction x="78.74" y="12.7"/>
 </segment>
 </net>
@@
 <pinref part="R10" gate="G$1" pin="1"/>
 <wire x1="78.74" y1="-7.62" x2="76.2" y2="-7.62" width="0.1524" layer="91"/>
-<wire x1="78.74" y1="2.54" x2="78.74" y2="-7.62" width="0.1524" layer="91"/>
+<wire x1="78.74" y1="-2.54" x2="78.74" y2="-7.62" width="0.1524" layer="91"/>
 <junction x="78.74" y="-7.62"/>
 </segment>
